File: piezoamp.brd (EAGLE design)
At the start: 36 x 41.5 mm, 20 parts, among them J3 OSTVN02A150, J5 OSTVN04A150, J6 OSTVN02A150, U1 968, U2 968, U3 AD8512

Commit message: Updates to README
- Also, added mounting holes to PCB
Parts:
- removed R5: 10k, jonnew:0603
- added RA: 1k, jonnew:0603
- C1, C2: value 0.1uF -> 68nF
- C3, C4: value 10nF -> 0.1uF
- R3: value 1k -> 10k
- moved R3 9.72 mm to (27.8, 9.51), turned to 0 degrees
- moved C1 7.53 mm to (15.2, 10.4)
- moved C3 7.53 mm to (20.7, 15.6)
- moved C2 3.06 mm to (14.7, 13.1), turned to 180 degrees
- moved C4 3.06 mm to (15.3, 16.1), turned to 270 degrees
- renumbered C5 to CF, R4 to RB, R40 to RF
Connections:
- net +15V0: now also C3.2, R3.1; no longer C1.2, R5.1
- net -15V0: now also C4.1; no longer C2.1
- net GND: now also C3.1; no longer C1.1
- net N$1: now also C2.1; no longer C4.1
- net N$2: now also RA.2; no longer R3.2
- net N$4: now also C1.1; no longer C3.1
- net N$7: now also R3.2; no longer R5.2
- net VOUT: now also C1.2, RA.1; no longer C3.2, R3.1
Routing:
- net BAT-: track 42.7 -> 44.1 mm
Other:
- board text added: "PIEZOFILM AMPLIFIER"
- board text removed: "PIEZO-FILM AMPLIFIER"

Commit message: Fixed circuit error and produced PCB gerbers
- Non inverting input of charge amplifer was not tied to ground
Connections:
- removed net IN-: J1.1, J1.2, J6.P$2, U3.3
- net GND: now also J1.1, J1.2, J6.P$2, U3.3
Routing:
- net GND: track 5.10 -> 33.0 mm, vias 4 -> 5
- net IN-: track 26.2 -> 0.00 mm
Other:
- board text added: "GND"

Commit message: Added mounting holes
- Few other minor tweaks
- New gerbers
Routing:
- net BAT-: track 44.1 -> 49.0 mm
- net GND: vias 5 -> 21
- added copper zone on layer 1, net GND
Changed lines of the file:
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@@
 <hole x="33.1" y="36.6" drill="3.5"/>
 <hole x="2.9" y="36.6" drill="3.5"/>
-<hole x="8.6" y="19.7" drill="3.5"/>
+<hole x="7.9" y="19.5" drill="3.5"/>
 </plain>
 <attributes>
@@
 <wire x1="17.6298" y1="18.1784" x2="17.6298" y2="16.5298" width="0.2032" layer="1"/>
 <wire x1="17.6298" y1="16.5298" x2="17.6" y2="16.5" width="0.2032" layer="1"/>
+<polygon width="0.2" layer="1" thermals="no">
+<vertex x="-2.2" y="-3.8"/>
+<vertex x="42" y="-3.8"/>
+<vertex x="42" y="39.7"/>
+<vertex x="-2.2" y="39.7"/>
+</polygon>
+<via x="11.5" y="20" extent="1-16" drill="0.35"/>
+<via x="7.6" y="13.3" extent="1-16" drill="0.35"/>
+<via x="1.5" y="9.1" extent="1-16" drill="0.35"/>
+<via x="1" y="17.9" extent="1-16" drill="0.35"/>
+<via x="1.3" y="28.2" extent="1-16" drill="0.35"/>
+<via x="9" y="37.5" extent="1-16" drill="0.35"/>
+<via x="18.5" y="37.3" extent="1-16" drill="0.35"/>
+<via x="18.7" y="31.9" extent="1-16" drill="0.35"/>
+<via x="29.4" y="36.5" extent="1-16" drill="0.35"/>
+<via x="34.5" y="32.2" extent="1-16" drill="0.35"/>
+<via x="34.5" y="13.5" extent="1-16" drill="0.35"/>
+<via x="34.8" y="5.1" extent="1-16" drill="0.35"/>
+<via x="15.5" y="-0.8" extent="1-16" drill="0.35"/>
+<via x="28" y="-0.6" extent="1-16" drill="0.35"/>
+<via x="2.3" y="-0.9" extent="1-16" drill="0.35"/>
+<via x="25.3" y="17.1" extent="1-16" drill="0.35"/>
 </signal>
 <signal name="+15V0">
@@
 <wire x1="10.6" y1="3.1" x2="10.6" y2="2.466" width="0.5" layer="16"/>
 <wire x1="10.6" y1="2.466" x2="11.8" y2="1.266" width="0.5" layer="16"/>
-<wire x1="5.2" y1="8.35" x2="8.3" y2="5.25" width="0.5" layer="1"/>
-<wire x1="11.15" y1="32.5" x2="5.2" y2="26.55" width="0.5" layer="1"/>
-<wire x1="5.2" y1="26.55" x2="5.2" y2="8.35" width="0.5" layer="1"/>
+<wire x1="8.3" y1="5.25" x2="3.3" y2="10.25" width="0.7" layer="1"/>
+<wire x1="5.6" y1="32.5" x2="11.15" y2="32.5" width="0.7" layer="1"/>
+<wire x1="3.3" y1="10.25" x2="3.3" y2="30.2" width="0.7" layer="1"/>
+<wire x1="3.3" y1="30.2" x2="5.6" y2="32.5" width="0.7" layer="1"/>
 </signal>
 <signal name="BAT+">

Commit message: Replaced JFET amp with inexpensive option
- Also produced final gerbers
- Send to fab
Parts:
- CF: value 10pF -> 22pF
- J3, J6: value OSTVN02A150 -> OSTVN02
- U3: value AD8512 -> ADTL082J; device jonnew:SOP65P490X110-8N -> jonnew:SOIC127P500X400-8N
- moved R1 2.50 mm to (14.8, 21.5)
- moved C3 2.10 mm to (22.8, 15.6)
- moved RF 1.84 mm to (22.8, 19.3), turned to 270 degrees
- moved U3 1.15 mm to (18.9, 16.4)
- moved CF 0.45 mm to (18.9, 21.5)
Routing:
- net GND: track 33.0 -> 3.94 mm, vias 21 -> 27
- net N$4: track 17.4 -> 14.4 mm
- net N$5: track 6.64 -> 9.42 mm
- net -15V0: track 22.0 -> 23.0 mm
- net IN+: track 20.9 -> 21.8 mm, vias 0 -> 2
- net +15V0: track 28.7 -> 27.7 mm
- net N$2: track 4.00 -> 4.62 mm
Other:
- board size 36 x 41.5 mm -> 39 x 41.5 mm
