File: piezoamp.sch (EAGLE design)
At the start: 20 parts, among them J3 OSTVN02A150, J5 OSTVN04A150, J6 OSTVN02A150, U1 968, U2 968, U3 AD8512

Commit message: Updates to README
- Also, added mounting holes to PCB
Parts:
- removed C5: 10pF, jonnew:C_0603
- removed R4: 1k, jonnew:R_0603
- removed R40: 100M, jonnew:R_0603
- removed R5: 10k, jonnew:R_0603
- added CF: 10pF, jonnew:C_0603
- added RA, RB: 1k, jonnew:R_0603
- added RF: 100M, jonnew:R_0603
- C1, C2: value 0.1uF -> 68nF
- C3, C4: value 10nF -> 0.1uF
- R3: value 1k -> 10k
Connections:
- net +15V0: now also C3.2, R3.1; no longer C1.2, R5.1
- net -15V0: now also C4.1; no longer C2.1
- net GND: now also C3.1, RB.2; no longer C1.1, R4.2
- net IN+: now also CF.1, RF.1; no longer C5.1, R40.1
- net N$1: now also C2.1; no longer C4.1
- net N$2: now also RA.2, RB.1; no longer R3.2, R4.1
- net N$4: now also C1.1; no longer C3.1
- net N$5: now also CF.2, RF.2; no longer C5.2, R40.2
- net N$7: now also R3.2; no longer R5.2
- net VOUT: now also C1.2, RA.1; no longer C3.2, R3.1
Other:
- moved on the sheet: C1, C2, C3, C4, J1, J3, J6, R1, R2, R3, U3G$1, U3G$2

Commit message: Fixed circuit error and produced PCB gerbers
- Non inverting input of charge amplifer was not tied to ground
Connections:
- removed net IN-: J1.1, J1.2, J6.2, U3G$1.+IN
- net GND: now also J1.1, J1.2, J6.2, U3G$1.+IN
Changed lines of the file:
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@@
 <junction x="-116.84" y="68.58"/>
+</segment>
+<segment>
+<pinref part="U3" gate="G$1" pin="+IN"/>
+<wire x1="-68.58" y1="-5.08" x2="-83.82" y2="-5.08" width="0.1524" layer="91"/>
+<wire x1="-83.82" y1="-5.08" x2="-83.82" y2="-22.86" width="0.1524" layer="91"/>
+<pinref part="SUPPLY5" gate="PE" pin="GND"/>
+<wire x1="-83.82" y1="-5.08" x2="-106.68" y2="-5.08" width="0.1524" layer="91"/>
+<junction x="-83.82" y="-5.08"/>
+<pinref part="J1" gate="G$1" pin="2"/>
+<pinref part="J1" gate="G$1" pin="1"/>
+<wire x1="-106.68" y1="-5.08" x2="-109.22" y2="-5.08" width="0.1524" layer="91"/>
+<wire x1="-109.22" y1="-7.62" x2="-106.68" y2="-7.62" width="0.1524" layer="91"/>
+<wire x1="-106.68" y1="-7.62" x2="-106.68" y2="-5.08" width="0.1524" layer="91"/>
+<junction x="-106.68" y="-5.08"/>
+<junction x="-106.68" y="-7.62"/>
+<wire x1="-106.68" y1="-7.62" x2="-106.68" y2="-12.7" width="0.1524" layer="91"/>
+<wire x1="-106.68" y1="-12.7" x2="-124.46" y2="-12.7" width="0.1524" layer="91"/>
+<wire x1="-124.46" y1="-12.7" x2="-124.46" y2="-5.08" width="0.1524" layer="91"/>
+<pinref part="J6" gate="G$1" pin="2"/>
+<wire x1="-124.46" y1="-5.08" x2="-129.54" y2="-5.08" width="0.1524" layer="91"/>
 </segment>
 </net>
@@
 </segment>
 </net>
-<net name="IN-" class="0">
-<segment>
-<pinref part="U3" gate="G$1" pin="+IN"/>
-<wire x1="-68.58" y1="-5.08" x2="-83.82" y2="-5.08" width="0.1524" layer="91"/>
-<wire x1="-83.82" y1="-5.08" x2="-83.82" y2="-22.86" width="0.1524" layer="91"/>
-<pinref part="SUPPLY5" gate="PE" pin="GND"/>
-<wire x1="-83.82" y1="-5.08" x2="-106.68" y2="-5.08" width="0.1524" layer="91"/>
-<junction x="-83.82" y="-5.08"/>
-<pinref part="J1" gate="G$1" pin="2"/>
-<pinref part="J1" gate="G$1" pin="1"/>
-<wire x1="-106.68" y1="-5.08" x2="-109.22" y2="-5.08" width="0.1524" layer="91"/>
-<wire x1="-109.22" y1="-7.62" x2="-106.68" y2="-7.62" width="0.1524" layer="91"/>
-<wire x1="-106.68" y1="-7.62" x2="-106.68" y2="-5.08" width="0.1524" layer="91"/>
-<junction x="-106.68" y="-5.08"/>
-<junction x="-106.68" y="-7.62"/>
-<wire x1="-106.68" y1="-7.62" x2="-106.68" y2="-12.7" width="0.1524" layer="91"/>
-<wire x1="-106.68" y1="-12.7" x2="-124.46" y2="-12.7" width="0.1524" layer="91"/>
-<wire x1="-124.46" y1="-12.7" x2="-124.46" y2="-5.08" width="0.1524" layer="91"/>
-<pinref part="J6" gate="G$1" pin="2"/>
-<wire x1="-124.46" y1="-5.08" x2="-129.54" y2="-5.08" width="0.1524" layer="91"/>
-</segment>
-</net>
 <net name="N$7" class="0">
 <segment>
@@
 </sheet>
 </sheets>
+<errors>
+</errors>
 </schematic>
 </drawing>

Commit message: Replaced JFET amp with inexpensive option
- Also produced final gerbers
- Send to fab
Parts:
- CF: value 10pF -> 22pF
- J3, J6: value OSTVN02A150 -> OSTVN02
- U3: value AD8512 -> ADTL082J; device jonnew:AD851_SOIC -> jonnew:DUAL-OPAMP_SOIC
Changed lines of the file:
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@@
 <?xml version="1.0" encoding="utf-8"?>
 <!DOCTYPE eagle SYSTEM "eagle.dtd">
-<eagle version="8.3.2">
+<eagle version="9.0.0">
 <drawing>
 <settings>
@@
 </classes>
 <parts>
-<part name="U3" library="jonnew" deviceset="AD851*" device="_SOIC" value="AD8512"/>
 <part name="C3" library="jonnew" deviceset="C" device="_0603" value="0.1uF"/>
 <part name="C4" library="jonnew" deviceset="C" device="_0603" value="0.1uF"/>
@@
 <part name="U9" library="jonnew" deviceset="+15V" device=""/>
 <part name="RB" library="jonnew" deviceset="R" device="_0603" value="1k"/>
-<part name="CF" library="jonnew" deviceset="C" device="_0603" value="10pF"/>
+<part name="CF" library="jonnew" deviceset="C" device="_0603" value="22pF"/>
 <part name="RF" library="jonnew" deviceset="R" device="_0603" value="100M"/>
 <part name="SUPPLY3" library="jonnew" deviceset="GND" device=""/>
@@
 <part name="U8" library="jonnew" deviceset="-15V" device=""/>
 <part name="SUPPLY8" library="jonnew" deviceset="GND" device=""/>
-<part name="J3" library="jonnew" deviceset="SCREW2" device="" value="OSTVN02A150"/>
+<part name="J3" library="jonnew" deviceset="SCREW2" device="" value="OSTVN02"/>
 <part name="S1" library="jonnew" deviceset="DPDT" device="_P040130" value="EG2210"/>
-<part name="J6" library="jonnew" deviceset="SCREW2" device="" value="OSTVN02A150"/>
+<part name="J6" library="jonnew" deviceset="SCREW2" device="" value="OSTVN02"/>
 <part name="J5" library="jonnew" deviceset="SCREW4" device="" value="OSTVN04A150"/>
 <part name="SUPPLY9" library="jonnew" deviceset="GND" device=""/>
 <part name="U$1" library="jonnew" deviceset="DOCFIELD-GEN" device=""/>
+<part name="U3" library="jonnew" deviceset="DUAL-OPAMP" device="_SOIC" value="ADTL082J"/>
 </parts>
 <sheets>
@@
 </plain>
 <instances>
-<instance part="U3" gate="G$1" x="-60.96" y="-2.54" rot="MR180"/>
-<instance part="U3" gate="G$2" x="15.24" y="-5.08"/>
-<instance part="U3" gate="G$3" x="12.7" y="-5.08"/>
 <instance part="C3" gate="C" x="22.86" y="7.62" rot="R270"/>
 <instance part="C4" gate="C" x="20.32" y="-17.78" rot="R90"/>
@@
 <instance part="SUPPLY9" gate="PE" x="-116.84" y="53.34"/>
 <instance part="U$1" gate="G$1" x="-152.4" y="-71.12"/>
+<instance part="U3" gate="G$1" x="-60.96" y="-2.54" rot="MR180"/>
+<instance part="U3" gate="G$2" x="15.24" y="-5.08"/>
+<instance part="U3" gate="G$3" x="12.7" y="-5.08"/>
 </instances>
 <busses>
@@
 <segment>
 <pinref part="R2" gate="R" pin="2"/>
-<pinref part="U3" gate="G$2" pin="+IN"/>
 <wire x1="-15.24" y1="-2.54" x2="-10.16" y2="-2.54" width="0.1524" layer="91"/>
 <pinref part="C2" gate="C" pin="1"/>
@@
 <wire x1="-10.16" y1="-22.86" x2="-10.16" y2="-2.54" width="0.1524" layer="91"/>
 <junction x="-10.16" y="-2.54"/>
+<pinref part="U3" gate="G$2" pin="+IN"/>
 </segment>
 </net>
@@
 <segment>
 <pinref part="U10" gate="G$1" pin="-15V0"/>
-<pinref part="U3" gate="G$3" pin="V-"/>
 <wire x1="15.24" y1="-22.86" x2="15.24" y2="-12.7" width="0.1524" layer="91"/>
 <pinref part="C4" gate="C" pin="1"/>
 <wire x1="15.24" y1="-12.7" x2="17.78" y2="-17.78" width="0.1524" layer="91"/>
+<pinref part="U3" gate="G$3" pin="V-"/>
 <junction x="15.24" y="-12.7"/>
 </segment>
@@
 </segment>
 <segment>
-<pinref part="U3" gate="G$1" pin="+IN"/>
 <wire x1="-68.58" y1="-5.08" x2="-83.82" y2="-5.08" width="0.1524" layer="91"/>
 <wire x1="-83.82" y1="-5.08" x2="-83.82" y2="-22.86" width="0.1524" layer="91"/>
@@
 <pinref part="J6" gate="G$1" pin="2"/>
 <wire x1="-124.46" y1="-5.08" x2="-129.54" y2="-5.08" width="0.1524" layer="91"/>
+<pinref part="U3" gate="G$1" pin="+IN"/>
 </segment>
 </net>
 <net name="+15V0" class="0">
 <segment>
-<pinref part="U3" gate="G$3" pin="V+"/>
 <pinref part="U9" gate="G$1" pin="+15V0"/>
 <wire x1="15.24" y1="2.54" x2="15.24" y2="10.16" width="0.1524" layer="91"/>
 <pinref part="C3" gate="C" pin="2"/>
 <wire x1="15.24" y1="2.54" x2="17.78" y2="7.62" width="0.1524" layer="91"/>
+<pinref part="U3" gate="G$3" pin="V+"/>
 <junction x="15.24" y="2.54"/>
 </segment>
@@
 <wire x1="2.54" y1="-40.64" x2="12.7" y2="-40.64" width="0.1524" layer="91"/>
 <wire x1="2.54" y1="-40.64" x2="2.54" y2="-43.18" width="0.1524" layer="91"/>
-<pinref part="U3" gate="G$2" pin="-IN"/>
 <wire x1="7.62" y1="-7.62" x2="2.54" y2="-7.62" width="0.1524" layer="91"/>
 <wire x1="2.54" y1="-7.62" x2="2.54" y2="-40.64" width="0.1524" layer="91"/>
 <junction x="2.54" y="-40.64"/>
+<pinref part="U3" gate="G$2" pin="-IN"/>
 </segment>
 </net>
@@
 <wire x1="22.86" y1="-40.64" x2="43.18" y2="-40.64" width="0.1524" layer="91"/>
 <wire x1="43.18" y1="-40.64" x2="43.18" y2="-5.08" width="0.1524" layer="91"/>
-<pinref part="U3" gate="G$2" pin="OUT"/>
 <wire x1="43.18" y1="-5.08" x2="22.86" y2="-5.08" width="0.1524" layer="91"/>
 <wire x1="43.18" y1="-5.08" x2="43.18" y2="25.4" width="0.1524" layer="91"/>
@@
 <wire x1="43.18" y1="-5.08" x2="71.12" y2="-5.08" width="0.1524" layer="91"/>
 <pinref part="J3" gate="G$1" pin="1"/>
+<pinref part="U3" gate="G$2" pin="OUT"/>
 </segment>
 </net>
@@
 <pinref part="RF" gate="R" pin="2"/>
 <wire x1="-43.18" y1="25.4" x2="-58.42" y2="25.4" width="0.1524" layer="91"/>
-<pinref part="U3" gate="G$1" pin="OUT"/>
 <wire x1="-43.18" y1="-2.54" x2="-53.34" y2="-2.54" width="0.1524" layer="91"/>
 <junction x="-43.18" y="-2.54"/>
+<pinref part="U3" gate="G$1" pin="OUT"/>
 </segment>
 </net>
 <net name="IN+" class="0">
 <segment>
-<pinref part="U3" gate="G$1" pin="-IN"/>
 <wire x1="-68.58" y1="0" x2="-83.82" y2="0" width="0.1524" layer="91"/>
 <wire x1="-83.82" y1="0" x2="-83.82" y2="12.7" width="0.1524" layer="91"/>
@@
 <wire x1="-119.38" y1="5.08" x2="-106.68" y2="5.08" width="0.1524" layer="91"/>
 <wire x1="-106.68" y1="5.08" x2="-106.68" y2="0" width="0.1524" layer="91"/>
-</segment>
-</net>
+<pinref part="U3" gate="G$1" pin="-IN"/>
+</segment>
+</net>
